File: hardware/Keyboard.kicad_pcb (KiCad board)
At the start: 2 copper layers, 306.6 x 115.2 mm, 190 parts, among them J1 USB_C_Receptacle_USB2.0_16P, SW1 SW_Push, SW2 SW_Push, U1 STM32F072CBTx, U2 XC6206PxxxMR

Commit message: finished routing --> need to add test points and add i2c display. also need to request a review and refine routing.
Parts:
- S27, S3, S56: footprint PCM_marbastlib-mx:STAB_MX_P_6.25u -> PCM_marbastlib-mx:STAB_MX_P_2u
- moved S3 293.2 mm to (23.7, 120.6)
- moved S75 199.3 mm to (133.2, 139.7)
- moved S27 193.2 mm to (266.5, 101.5)
- moved S56 139.2 mm to (268.9, 63.4)
- moved R5 3.64 mm to (275.3, 37.7), turned to 180 degrees
- moved C5 0.39 mm to (262.7, 50.1)
- moved C7 0.39 mm to (261.1, 50.1)
- moved D86 0.14 mm to (287.0, 36.4)
Connections:
- U1 pad 10: unconnected-(U1-PA0-Pad10) -> col10
- U1 pad 11: unconnected-(U1-PA1-Pad11) -> col11
- U1 pad 12: unconnected-(U1-PA2-Pad12) -> col12
- U1 pad 28: unconnected-(U1-PB15-Pad28) -> row0
- U1 pad 3: unconnected-(U1-PC14-Pad3) -> col15
- U1 pad 39: unconnected-(U1-PB3-Pad39) -> row5
- U1 pad 40: unconnected-(U1-PB4-Pad40) -> row4
- U1 pad 41: unconnected-(U1-PB5-Pad41) -> row3
- U1 pad 45: unconnected-(U1-PB8-Pad45) -> row2
- U1 pad 46: unconnected-(U1-PB9-Pad46) -> row1
- U1 pad 5: unconnected-(U1-PF0-Pad5) -> col14
- U1 pad 6: unconnected-(U1-PF1-Pad6) -> col13
Routing:
- net row5: track 283.4 -> 397.6 mm
- net row4: track 273.8 -> 367.8 mm, vias 0 -> 2
- net row3: track 278.6 -> 360.4 mm, vias 0 -> 2
- net col10: track 124.9 -> 191.1 mm, vias 0 -> 1
- net row2: track 281.0 -> 333.5 mm, vias 0 -> 2
- net col11: track 123.7 -> 169.6 mm, vias 0 -> 2
- net col13: track 64.1 -> 108.5 mm, vias 0 -> 1
- net col15: track 76.2 -> 114.2 mm, vias 0 -> 1
- net GND: track 30.1 -> 62.5 mm, vias 2 -> 10
- net row1: track 285.8 -> 315.0 mm, vias 0 -> 4
- net col12: track 118.5 -> 143.6 mm, vias 0 -> 2
- net row0: track 228.6 -> 253.6 mm, vias 0 -> 10
- net col14: track 86.7 -> 101.4 mm, vias 0 -> 1
- net unconnected-(U1-PB6-Pad42): track 0.00 -> 7.38 mm
- net unconnected-(U1-PB7-Pad43): track 0.00 -> 6.97 mm
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Other:
- board size 306.6 x 115.2 mm -> 306.6 x 118 mm
