File: hardware/Keyboard.kicad_pcb (KiCad board)
At the start: 2 copper layers, 306.6 x 117.8 mm, 191 parts, among them J1 USB_C_Receptacle_USB2.0_16P, J2 Conn_01x04, SW1 SW_Push, SW2 SW_Push, U1 STM32F072CBTx, U2 XC6206PxxxMR

Commit message: added testpoints, need to readd library
Parts:
- added 3.3vTP1: TestPoint, TestPoint:TestPoint_Pad_2.0x2.0mm, B.Cu at (288.8, 51.5)
- added 3.3vTP2: TestPoint, TestPoint:TestPoint_Pad_2.0x2.0mm, B.Cu at (251.8, 51.8)
- added 5vTP1: TestPoint, TestPoint:TestPoint_Pad_2.0x2.0mm, B.Cu at (288.8, 46.0)
- added GNDTP1: TestPoint, TestPoint:TestPoint_Pad_2.0x2.0mm, B.Cu at (242.0, 52.0)
- added GNDTP2: TestPoint, TestPoint:TestPoint_Pad_2.0x2.0mm, B.Cu at (303.0, 70.5)
- added J3: Conn_01x04, Connector_PinHeader_2.54mm:PinHeader_1x04_P2.54mm_Vertical, F.Cu at (303.1, 51.5)
- added OL1: OLED, kbd:OLED, F.Cu at (300.4, 43.2)
- added R6: 5.1k, Resistor_SMD:R_0603_1608Metric_Pad0.98x0.95mm_HandSolder, B.Cu at (303.6, 44.4)
- added R7: 5.1k, Resistor_SMD:R_0603_1608Metric_Pad0.98x0.95mm_HandSolder, B.Cu at (303.6, 47.0)
- added TP1: col0, TestPoint:TestPoint_Pad_2.0x2.0mm, B.Cu at (7.80, 70.2)
- added TP10: col1, TestPoint:TestPoint_Pad_2.0x2.0mm, B.Cu at (176.2, 70.2)
- added TP11: col0, TestPoint:TestPoint_Pad_2.0x2.0mm, B.Cu at (194.6, 70.6)
- added TP12: col1, TestPoint:TestPoint_Pad_2.0x2.0mm, B.Cu at (213.2, 70.4)
- added TP13: col0, TestPoint:TestPoint_Pad_2.0x2.0mm, B.Cu at (233.2, 70.2)
- added TP14: col1, TestPoint:TestPoint_Pad_2.0x2.0mm, B.Cu at (248.2, 70.2)
- added TP15: col0, TestPoint:TestPoint_Pad_2.0x2.0mm, B.Cu at (266.0, 70.2)
- added TP16: col1, TestPoint:TestPoint_Pad_2.0x2.0mm, B.Cu at (293.8, 70.2)
- added TP17: col1, TestPoint:TestPoint_Pad_2.0x2.0mm, B.Cu at (251.8, 47.4)
- added TP18: col0, TestPoint:TestPoint_Pad_2.0x2.0mm, B.Cu at (256.2, 66.4)
- added TP19: col1, TestPoint:TestPoint_Pad_2.0x2.0mm, B.Cu at (259.2, 85.4)
- added TP2: col1, TestPoint:TestPoint_Pad_2.0x2.0mm, B.Cu at (27.6, 70.0)
- added TP20: col0, TestPoint:TestPoint_Pad_2.0x2.0mm, B.Cu at (259.4, 104.6)
- added TP21: col1, TestPoint:TestPoint_Pad_2.0x2.0mm, B.Cu at (259.6, 123.4)
- added TP22: col1, TestPoint:TestPoint_Pad_2.0x2.0mm, B.Cu at (268.8, 142.6)
- added TP3: col0, TestPoint:TestPoint_Pad_2.0x2.0mm, B.Cu at (42.8, 70.0)
- added TP4: col1, TestPoint:TestPoint_Pad_2.0x2.0mm, B.Cu at (61.6, 70.0)
- added TP5: col0, TestPoint:TestPoint_Pad_2.0x2.0mm, B.Cu at (80.6, 69.8)
- added TP6: col1, TestPoint:TestPoint_Pad_2.0x2.0mm, B.Cu at (99.2, 70.0)
- added TP7: col0, TestPoint:TestPoint_Pad_2.0x2.0mm, B.Cu at (118.8, 69.8)
- added TP8: col1, TestPoint:TestPoint_Pad_2.0x2.0mm, B.Cu at (138.4, 70.2)
- added TP9: col0, TestPoint:TestPoint_Pad_2.0x2.0mm, B.Cu at (157.0, 70.2)
- added VBUSTP1: TestPoint, TestPoint:TestPoint_Pad_2.0x2.0mm, B.Cu at (303.2, 38.2)
- renumbered C9 to C1, C6 to C10, C7 to C11, C10 to C2, C1 to C3, C2 to C4, C8 to C5, C11 to C6, C3 to C7, C4 to C8, C5 to C9, D86 to D1, D15 to D10, D45 to D11, D73 to D12, D3 to D13, D16 to D14, D30 to D15, D46 to D16, D59 to D17, D74 to D18, D4 to D19, D85 to D2, D17 to D20, D31 to D21, D47 to D22, D60 to D23, D5 to D24, D18 to D25, D32 to D26, D48 to D27, D61 to D28, D6 to D29, D1 to D3, D19 to D30, D33 to D31, D49 to D32, D62 to D33, D7 to D34, D20 to D35, D34 to D36, D50 to D37, D63 to D38, D8 to D39, D14 to D4, D21 to D40, D35 to D41, D51 to D42, D64 to D43, D75 to D44, D9 to D45, D22 to D46, D36 to D47, D52 to D48, D65 to D49, D29 to D5, D10 to D50, D23 to D51, D37 to D52, D66 to D54, D11 to D55, D24 to D56, D38 to D57, D54 to D58, D67 to D59, D44 to D6, D76 to D60, D12 to D61, D25 to D62, D39 to D63, D55 to D64, D68 to D65, D77 to D66, D13 to D67, D26 to D68, D40 to D69, D58 to D7, D69 to D70, D78 to D71, D41 to D72, D79 to D73, D27 to D74, D42 to D75, D56 to D76, D70 to D77, D80 to D78, D28 to D79, D72 to D8, D43 to D80, D57 to D81, D71 to D82, D81 to D83, D2 to D9, MX73 to MX10, MX3 to MX11, MX16 to MX12, MX30 to MX13, MX46 to MX14, MX59 to MX15, MX74 to MX16, MX4 to MX17, MX17 to MX18, MX31 to MX19, MX14 to MX2, MX47 to MX20, MX60 to MX21, MX5 to MX22, MX18 to MX23, MX32 to MX24, MX48 to MX25, MX61 to MX26, MX6 to MX27, MX19 to MX28, MX33 to MX29, MX29 to MX3, MX49 to MX30, MX62 to MX31, MX7 to MX32, MX20 to MX33, MX50 to MX35, MX63 to MX36, MX8 to MX37, MX21 to MX38, MX35 to MX39, MX44 to MX4, MX51 to MX40, MX64 to MX41, MX75 to MX42, MX9 to MX43, MX22 to MX44, MX36 to MX45, MX52 to MX46, MX65 to MX47, MX10 to MX48, MX23 to MX49, MX58 to MX5, MX37 to MX50, MX53 to MX51, MX66 to MX52, MX11 to MX53, MX24 to MX54, MX38 to MX55, MX54 to MX56, MX67 to MX57, MX76 to MX58, MX12 to MX59, MX72 to MX6, MX25 to MX60, MX39 to MX61, MX55 to MX62, MX68 to MX63, MX77 to MX64, MX13 to MX65, MX26 to MX66, MX40 to MX67, MX69 to MX68, MX78 to MX69, MX2 to MX7, MX41 to MX70, MX79 to MX71, MX27 to MX72, MX42 to MX73, MX56 to MX74, MX70 to MX75, MX80 to MX76, MX28 to MX77, MX43 to MX78, MX57 to MX79, MX15 to MX8, MX71 to MX80, MX45 to MX9, R4 to R1, R5 to R2, R1 to R3, R3 to R4, R2 to R5, S3 to S1, S75 to S2, S27 to S3, S56 to S4, SW2 to SW1, SW1 to SW2, U2 to U1, U1 to U2
Routing:
- net /SCL: track 7.38 -> 44.9 mm, vias 0 -> 1
- net /SDA: track 6.97 -> 43.6 mm, vias 0 -> 1
- net /VBUS: track 13.4 -> 22.2 mm
- net +3.3V: track 27.6 -> 35.2 mm, vias 8 -> 10
- net +5V: track 8.09 -> 11.6 mm
- net col9: vias 1 -> 2
- net col8: vias 1 -> 2
- net col7: vias 1 -> 2
- net col11: vias 2 -> 3
- net col6: vias 1 -> 2
- net col5: vias 1 -> 2
- net col4: vias 0 -> 1
- net col3: vias 0 -> 1
- net col2: vias 0 -> 1
- net col15: vias 1 -> 2
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Other:
- board text added: "3.3v"
