File: hardware/Keyboard.kicad_pcb (KiCad board)
At the start: 2 copper layers, 306.6 x 117.8 mm, 223 parts, among them J1 USB_C_Receptacle_USB2.0_16P, J2 Conn_01x04, J3 Conn_01x04, SW1 SW_Push, SW2 SW_Push, U1 XC6206PxxxMR, U2 STM32F072CBTx

Commit message: production files added --> ready for assembly
Parts:
- removed the D1 at (287.0, 36.4)
- added G***: LOGO, footprints:blossoms100, F.Cu at (43.9, 83.8)
- added G***: LOGO, footprints:f17, F.Cu at (152.7, 93.0)
- added H1: MountingHole, MountingHole:MountingHole_3.2mm_M3_ISO7380, F.Cu at (4.25, 94.8)
- added H2: MountingHole, MountingHole:MountingHole_3.2mm_M3_ISO7380, F.Cu at (96.0, 147.5)
- added H3: MountingHole, MountingHole:MountingHole_3.2mm_M3_ISO7380, F.Cu at (154.8, 54.0)
- added H4: MountingHole, MountingHole:MountingHole_3.2mm_M3_ISO7380, F.Cu at (303.5, 37.0)
- added H5: MountingHole, MountingHole:MountingHole_3.2mm_M3_ISO7380, F.Cu at (21.0, 53.8)
- added H6: MountingHole, MountingHole:MountingHole_3.2mm_M3_ISO7380, F.Cu at (173.5, 147.5)
- added H7: MountingHole, MountingHole:MountingHole_3.2mm_M3_ISO7380, F.Cu at (250.5, 45.5)
- added TP23: TestPoint, TestPoint:TestPoint_THTPad_1.0x1.0mm_Drill0.5mm, F.Cu at (279.6, 35.7)
- added TP24: TestPoint, TestPoint:TestPoint_THTPad_1.0x1.0mm_Drill0.5mm, F.Cu at (279.6, 37.7)
- added U3: USBLC6-2P6, Package_TO_SOT_SMD:SOT-666, B.Cu at (286.6, 37.0)
- J1: footprint PCM_marbastlib-various:USB_C_Receptacle_HRO_TYPE-C-31-M-23 -> Connector_USB:USB_C_Receptacle_GCT_USB4105-xx-A_16P_TopMnt_Horizontal
- VBUSTP1: moved to F.Cu
- moved TP17 21.1 mm to (230.8, 47.5)
- moved VBUSTP1 7.56 mm to (295.7, 37.9), turned to 0 degrees
- moved TP21 3.40 mm to (263.0, 123.2)
- moved C1 2.67 mm to (286.0, 39.8), turned to 180 degrees
- moved R3 2.27 mm to (297.2, 43.4)
- moved F1 2.11 mm to (287.8, 41.5)
- moved R5 1.67 mm to (292.2, 43.1)
- moved J1 0.48 mm to (294.6, 37.2)
- moved C2 0.05 mm to (287.8, 43.1)
- renumbered D3 to D1, D45 to D10, D50 to D11, D55 to D12, D61 to D13, D67 to D14, D4 to D15, D10 to D16, D14 to D17, D20 to D18, D25 to D19, D30 to D20, D35 to D21, D40 to D22, D46 to D23, D51 to D24, D56 to D25, D62 to D26, D68 to D27, D74 to D28, D79 to D29, D9 to D3, D5 to D30, D15 to D31, D21 to D32, D26 to D33, D31 to D34, D36 to D35, D41 to D36, D47 to D37, D52 to D38, D57 to D39, D13 to D4, D63 to D40, D69 to D41, D72 to D42, D75 to D43, D80 to D44, D6 to D45, D11 to D46, D16 to D47, D22 to D48, D27 to D49, D19 to D5, D32 to D50, D37 to D51, D42 to D52, D48 to D53, D53 to D54, D58 to D55, D64 to D56, D76 to D57, D81 to D58, D7 to D59, D24 to D6, D17 to D60, D23 to D61, D28 to D62, D33 to D63, D38 to D64, D43 to D65, D49 to D66, D54 to D67, D59 to D68, D65 to D69, D29 to D7, D77 to D71, D82 to D72, D8 to D73, D12 to D74, D18 to D75, D44 to D76, D60 to D77, D66 to D78, D71 to D79, D34 to D8, D73 to D80, D78 to D81, D83 to D82, D39 to D9, MX48 to MX10, MX53 to MX11, MX59 to MX12, MX65 to MX13, MX2 to MX14, MX8 to MX15, MX12 to MX16, MX18 to MX17, MX23 to MX18, MX28 to MX19, MX7 to MX2, MX33 to MX20, MX38 to MX21, MX44 to MX22, MX49 to MX23, MX54 to MX24, MX60 to MX25, MX66 to MX26, MX72 to MX27, MX77 to MX28, MX3 to MX29, MX11 to MX3, MX13 to MX30, MX19 to MX31, MX24 to MX32, MX29 to MX33, MX39 to MX35, MX45 to MX36, MX50 to MX37, MX55 to MX38, MX61 to MX39, MX17 to MX4, MX67 to MX40, MX70 to MX41, MX73 to MX42, MX78 to MX43, MX4 to MX44, MX9 to MX45, MX14 to MX46, MX20 to MX47, MX25 to MX48, MX30 to MX49, MX22 to MX5, MX35 to MX50, MX40 to MX51, MX46 to MX52, MX51 to MX53, MX56 to MX54, MX62 to MX55, MX74 to MX56, MX79 to MX57, MX5 to MX58, MX15 to MX59, MX27 to MX6, MX21 to MX60, MX26 to MX61, MX31 to MX62, MX36 to MX63, MX41 to MX64, MX47 to MX65, MX52 to MX66, MX57 to MX67, MX63 to MX68, MX68 to MX69, MX32 to MX7, MX75 to MX70, MX80 to MX71, MX6 to MX72, MX10 to MX73, MX16 to MX74, MX42 to MX75, MX58 to MX76, MX64 to MX77, MX69 to MX78, MX71 to MX79, MX37 to MX8, MX76 to MX80, MX43 to MX9, S3 to S1, S4 to S2, S1 to S3, S2 to S4
Connections:
- U2 pad 29: unconnected-(U2-PA8-Pad29) -> /Debug1
- U2 pad 30: unconnected-(U2-PA9-Pad30) -> /Debug2
- U2 pad 32: /D- -> /mcu_D-
- U2 pad 33: /D+ -> /mcu_D+
Routing:
- net /mcu_D+: track 0.00 -> 27.1 mm
- net /mcu_D-: track 0.00 -> 27.0 mm
- net /D-: track 39.9 -> 13.4 mm
- net /D+: track 37.0 -> 15.8 mm, vias 0 -> 2
- net GND: track 70.6 -> 86.2 mm
- net /VBUS: track 22.2 -> 20.0 mm
- net row0: track 253.6 -> 255.8 mm
- net /SCL: track 44.9 -> 47.0 mm
- net col0: track 366.4 -> 364.3 mm
- net Net-(J1-CC2): track 1.63 -> 2.52 mm
- net /SDA: track 43.6 -> 44.4 mm
- net col10: track 191.1 -> 190.4 mm
- net +5V: track 11.6 -> 11.0 mm
- net +3.3V: track 35.2 -> 34.6 mm
Other:
- board text added: "GND"
- board text added: "January 2026"
- board text added: "Karthik Kurapati"
- board text added: "Revision A"
- board text added: "SCL"
- board text added: "SDA"
- board text added: "SWCLK"
- board text added: "SWDIO"
- board text added: "col0"
- board text added: "col1"
- board text added: "col10"
- board text added: "col11"
- board text added: "col12"
- board text added: "col13"
- board text added: "col14"
- board text added: "col15"
- board text added: "col2"
- board text added: "col3"
- board text added: "col4"
- board text added: "col5"
- board text added: "col6"
- board text added: "col7"
- board text added: "col8"
- board text added: "col9"
